Commit message: Add files via upload

File: car_model.urdf (robot description, URDF)
Before this commit: robot car_model, 11 links, 10 joints
Links:
- link base_link: geometry collision box size=1.8 1.2 0.2; visual box size=1.8 1.2 0.2
Joints:
- joint hokuyo_joint: origin xyz=2.5 0 -0.5 rpy=0 0 0 -> xyz=2.1 0 -0.5 rpy=0 0 0
- joint left_steer_joint: origin xyz=2.4 -0.8 -0.25 rpy=0 0 0 -> xyz=1.8 -0.8 -0.25 rpy=0 0 0
- joint right_steer_joint: origin xyz=2.4 0.8 -0.25 rpy=0 0 0 -> xyz=1.8 0.8 -0.25 rpy=0 0 0
- joint steer_joint: origin xyz=2.4 0 -0.25 rpy=0 0 0 -> xyz=1.8 0 -0.25 rpy=0 0 0
